File: hardware/familamp.brd (EAGLE design)
At the start: 41.9 x 48.3 mm, 12 parts

Commit message: Final Board Design (I HOPE)
Parts:
- moved DC 1.27 mm to (5.08, 0.00)
Routing:
- net VCC: track 55.6 -> 56.4 mm
Changed lines of the file:
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@@
 <text x="13.97" y="16.51" size="1.27" layer="21" font="vector" ratio="15" rot="R270" align="bottom-center">by Jerad Jacob</text>
 <text x="-71.12" y="44.45" size="1.778" layer="51" font="vector" ratio="15">Jerad Jacob</text>
-<text x="2.921" y="0.254" size="0.8128" layer="23">5VDC 2A</text>
 <text x="26.67" y="24.13" size="1.27" layer="22" font="vector" rot="MR270" align="center">May the road rise up to meet you.
 May the wind always be at your back.
@@
 <wire x1="41.91" y1="48.26" x2="41.91" y2="0" width="0.254" layer="20"/>
 <wire x1="41.91" y1="0" x2="0" y2="0" width="0.254" layer="20"/>
+<text x="7.62" y="13.97" size="0.8128" layer="21" font="vector">5VDC 2A</text>
 </plain>
 <attributes>
@@
 <element name="U$2" library="SparkFun-Boards" package="LOGIC_LEVEL_CONVERTER" value="LOGIC_LEVEL_CONVERTER" x="2.54" y="25.4"/>
 <element name="R2" library="SparkFun-Resistors" package="AXIAL-0.4" value="" x="39.37" y="22.86" rot="R90"/>
-<element name="DC" library="SparkFun-Connectors" package="POWER_JACK_PTH" value="POWER_JACKPTH" x="5.08" y="1.27">
-<attribute name="PROD_ID" value="CONN-08197" x="5.08" y="1.27" size="1.778" layer="27" display="off"/>
+<element name="DC" library="SparkFun-Connectors" package="POWER_JACK_PTH" value="POWER_JACKPTH" x="5.08" y="0">
+<attribute name="PROD_ID" value="CONN-08197" x="5.08" y="0" size="1.778" layer="27" display="off"/>
 </element>
 <element name="J1" library="SparkFun-Connectors" package="1X03" value="" x="39.37" y="31.75" rot="R90"/>
@@
 <wire x1="19.05" y1="35.56" x2="17.78" y2="36.068" width="0.254" layer="1" curve="-43.602819"/>
 <wire x1="13.97" y1="34.29" x2="17.78" y2="36.068" width="0.254" layer="1" curve="50.033779"/>
-<wire x1="5.08" y1="14.97" x2="7.89" y2="16.51" width="0.254" layer="1" curve="-90"/>
+<wire x1="5.08" y1="13.7" x2="7.89" y2="16.51" width="0.254" layer="1" curve="-90"/>
 <wire x1="7.89" y1="16.51" x2="10.16" y2="16.51" width="0.254" layer="1"/>
 </signal>
